File: hardware/seeq.kicad_sch (KiCad schematic)
At the start: 87 parts, among them J1 MIDI IN, J2 AudioJack2_SwitchT, J3 Conn_01x06, J4 Conn_01x04, J5 AudioJack2_SwitchT, J6 MIDI OUT, SW1 SW_DIP_x01, SW10 SW_DIP_x01, SW11 SW_DIP_x01, SW12 SW_DIP_x01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

Commit message: Update software for PCB + PCB fixes
Parts:
- removed D34, D35, D36, D37: WS2812, LED_SMD:LED_WS2812_PLCC6_5.0x5.0mm_P1.6mm, symbol LED:WS2812
- added D34, D35, D36, D37: WS2812B, LED_SMD:LED_WS2812B_PLCC4_5.0x5.0mm_P3.2mm, symbol LED:WS2812B
Connections:
- net +3V3: now also D34.1 (VDD), D35.1 (VDD), D36.1 (VDD), D37.1 (VDD)
- net GND: now also D34.3 (VSS), D35.3 (VSS), D36.3 (VSS), D37.3 (VSS)
- net LED: now also D34.4 (DIN)
- net SCL: now also U2.27 (GPIO21); no longer U2.26 (GPIO20)
- net SDA: now also U2.26 (GPIO20); no longer U2.27 (GPIO21)
- new net: D36.2 (DOUT), D37.4 (DIN)
- new net: D35.2 (DOUT), D36.4 (DIN)
- new net: D34.2 (DOUT), D35.4 (DIN)

Commit message: Add kibot and docs
Parts:
- removed J2, J5: AudioJack2_SwitchT, Connector_Audio:Jack_3.5mm_CUI_SJ1-3533NG_Horizontal_CircularHoles, symbol Connector:AudioJack2_SwitchT
- added C1: 1uF, Capacitor_THT:C_Disc_D5.0mm_W2.5mm_P5.00mm, symbol Device:C
- added D38, D39, D40, D41, D42, D43: WS2812B, LED_SMD:LED_WS2812B_PLCC4_5.0x5.0mm_P3.2mm, symbol LED:WS2812B
- added J2, J5: AudioJack2, Keebio-Parts:TRRS-PJ-320A-no-Fmask, symbol Connector:AudioJack2
Connections:
- net +3V3: no longer D34.1 (VDD), D35.1 (VDD), D36.1 (VDD), D37.1 (VDD)
- net +5V: now also D34.1 (VDD), D35.1 (VDD), D36.1 (VDD), D37.1 (VDD), C1.1, D38.1 (VDD), D39.1 (VDD), D40.1 (VDD), D41.1 (VDD), D42.1 (VDD), D43.1 (VDD)
- net GND: now also C1.2, D38.3 (VSS), D39.3 (VSS), D40.3 (VSS), D41.3 (VSS), D42.3 (VSS), D43.3 (VSS), J5.T
- net at D37.2 (DOUT): now also D38.4 (DIN)
- net at U2.24 (GPIO18): now also J5.S
- net at J3.2 (Pin_2): now also J2.S
- net at J3.1 (Pin_1): now also J2.T
- new net: D40.2 (DOUT), D41.4 (DIN)
- new net: D39.2 (DOUT), D40.4 (DIN)
- new net: D38.2 (DOUT), D39.4 (DIN)
- new net: D41.2 (DOUT), D42.4 (DIN)
- new net: D42.2 (DOUT), D43.4 (DIN)
Other:
- title: (none) -> SEEQ Midi sequencer
- moved on the sheet: D34, D35, D36, D37

Commit message: fix erc / drc
Other:
- company: (none) -> Six Pixels
Changed lines of the file:
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@@
     (title "SEEQ Midi sequencer")
     (date "2023-02-09")
-    (rev "V1.0")
+    (rev "${VERSION}")
+    (company "Six Pixels")
   )
   (junction (at 13.97 59.69) (diameter 0) (color 0 0 0 0)
@@
   (junction (at 44.45 62.23) (diameter 0) (color 0 0 0 0)
   )
+  (junction (at 274.32 52.07) (diameter 0) (color 0 0 0 0)
+  )
   (junction (at 189.23 72.39) (diameter 0) (color 0 0 0 0)
   )
@@
   (junction (at 172.72 99.06) (diameter 0) (color 0 0 0 0)
   )
+  (junction (at 222.25 57.15) (diameter 0) (color 0 0 0 0)
+  )
   (junction (at 59.69 171.45) (diameter 0) (color 0 0 0 0)
   )
@@
   (junction (at 153.67 95.25) (diameter 0) (color 0 0 0 0)
   )
+  (junction (at 276.86 62.23) (diameter 0) (color 0 0 0 0)
+  )
   (junction (at 113.03 191.77) (diameter 0) (color 0 0 0 0)
   )
@@
     (stroke (width 0) (type default) (color 0 0 0 0))
   )
+  (wire (pts (xy 274.32 52.07) (xy 281.94 52.07))
+    (stroke (width 0) (type default) (color 0 0 0 0))
+  )
   (wire (pts (xy 134.62 45.72) (xy 134.62 72.39))
     (stroke (width 0) (type default) (color 0 0 0 0))
@@
     (stroke (width 0) (type default) (color 0 0 0 0))
   )
-  (wire (pts (xy 271.78 62.23) (xy 279.4 62.23))
+  (wire (pts (xy 271.78 62.23) (xy 276.86 62.23))
     (stroke (width 0) (type default) (color 0 0 0 0))
   )
@@
     (stroke (width 0) (type default) (color 0 0 0 0))
   )
-  (wire (pts (xy 271.78 52.07) (xy 276.86 52.07))
+  (wire (pts (xy 271.78 52.07) (xy 274.32 52.07))
     (stroke (width 0) (type default) (color 0 0 0 0))
   )
@@
     (stroke (width 0) (type default) (color 0 0 0 0))
   )
+  (wire (pts (xy 276.86 62.23) (xy 283.21 62.23))
+    (stroke (width 0) (type default) (color 0 0 0 0))
+  )
   (wire (pts (xy 171.45 45.72) (xy 172.72 45.72))
     (stroke (width 0) (type default) (color 0 0 0 0))
@@
     (stroke (width 0) (type default) (color 0 0 0 0))
   )
-  (wire (pts (xy 236.22 57.15) (xy 219.71 57.15))
+  (wire (pts (xy 236.22 57.15) (xy 222.25 57.15))
     (stroke (width 0) (type default) (color 0 0 0 0))
   )
@@
     (stroke (width 0) (type default) (color 0 0 0 0))
   )
+  (wire (pts (xy 222.25 57.15) (xy 219.71 57.15))
+    (stroke (width 0) (type default) (color 0 0 0 0))
+  )
   (wire (pts (xy 199.39 80.01) (xy 199.39 144.78))
     (stroke (width 0) (type default) (color 0 0 0 0))
@@
     (pin "2")
   )
+  (symbol (lib_id "power:PWR_FLAG") (at 276.86 62.23 0) (unit 1)
+    (in_bom yes) (on_board yes) (fields_autoplaced)
+    (property "Reference" "#FLG0102" (id 0) (at 276.86 60.325 0)
+      (effects (font (size 1.27 1.27)) hide)
+    )
+    (property "Value" "PWR_FLAG" (id 1) (at 276.86 58.6542 0))
+    (property "Footprint" "" (id 2) (at 276.86 62.23 0)
+      (effects (font (size 1.27 1.27)) hide)
+    )
+    (property "Datasheet" "~" (id 3) (at 276.86 62.23 0)
+      (effects (font (size 1.27 1.27)) hide)
+    )
+    (pin "1")
+  )
   (symbol (lib_id "power:GND") (at 252.73 127 0) (unit 1)
     (in_bom yes) (on_board yes) (fields_autoplaced)
@@
     (pin "2")
   )
-  (symbol (lib_id "power:+5V") (at 276.86 52.07 0) (unit 1)
+  (symbol (lib_id "power:+5V") (at 281.94 52.07 0) (unit 1)
     (in_bom yes) (on_board yes) (fields_autoplaced)
-    (property "Reference" "#PWR0114" (id 0) (at 276.86 55.88 0)
+    (property "Reference" "#PWR0114" (id 0) (at 281.94 55.88 0)
       (effects (font (size 1.27 1.27)) hide)
     )
-    (property "Value" "+5V" (id 1) (at 276.86 48.4942 0))
-    (property "Footprint" "" (id 2) (at 276.86 52.07 0)
+    (property "Value" "+5V" (id 1) (at 281.94 48.4942 0))
+    (property "Footprint" "" (id 2) (at 281.94 52.07 0)
       (effects (font (size 1.27 1.27)) hide)
     )
-    (property "Datasheet" "" (id 3) (at 276.86 52.07 0)
+    (property "Datasheet" "" (id 3) (at 281.94 52.07 0)
       (effects (font (size 1.27 1.27)) hide)
     )
@@
     (pin "2")
   )
+  (symbol (lib_id "power:PWR_FLAG") (at 222.25 57.15 0) (unit 1)
+    (in_bom yes) (on_board yes) (fields_autoplaced)
+    (property "Reference" "#FLG0101" (id 0) (at 222.25 55.245 0)
+      (effects (font (size 1.27 1.27)) hide)
+    )
+    (property "Value" "PWR_FLAG" (id 1) (at 222.25 53.5742 0))
+    (property "Footprint" "" (id 2) (at 222.25 57.15 0)
+      (effects (font (size 1.27 1.27)) hide)
+    )
+    (property "Datasheet" "~" (id 3) (at 222.25 57.15 0)
+      (effects (font (size 1.27 1.27)) hide)
+    )
+    (pin "1")
+  )
   (symbol (lib_id "power:+5V") (at 25.4 156.21 0) (unit 1)
     (in_bom yes) (on_board yes) (fields_autoplaced)
@@
     (pin "1")
   )
-  (symbol (lib_id "power:+3V3") (at 279.4 62.23 0) (unit 1)
+  (symbol (lib_id "power:+3V3") (at 283.21 62.23 0) (unit 1)
     (in_bom yes) (on_board yes) (fields_autoplaced)
-    (property "Reference" "#PWR0115" (id 0) (at 279.4 66.04 0)
+    (property "Reference" "#PWR0115" (id 0) (at 283.21 66.04 0)
       (effects (font (size 1.27 1.27)) hide)
     )
-    (property "Value" "+3V3" (id 1) (at 279.4 58.6542 0))
-    (property "Footprint" "" (id 2) (at 279.4 62.23 0)
+    (property "Value" "+3V3" (id 1) (at 283.21 58.6542 0))
+    (property "Footprint" "" (id 2) (at 283.21 62.23 0)
       (effects (font (size 1.27 1.27)) hide)
     )
-    (property "Datasheet" "" (id 3) (at 279.4 62.23 0)
+    (property "Datasheet" "" (id 3) (at 283.21 62.23 0)
       (effects (font (size 1.27 1.27)) hide)
     )
@@
     (pin "2")
   )
+  (symbol (lib_id "power:PWR_FLAG") (at 274.32 52.07 0) (unit 1)
+    (in_bom yes) (on_board yes) (fields_autoplaced)
+    (property "Reference" "#FLG0103" (id 0) (at 274.32 50.165 0)
+      (effects (font (size 1.27 1.27)) hide)
+    )
+    (property "Value" "PWR_FLAG" (id 1) (at 274.32 48.4942 0))
+    (property "Footprint" "" (id 2) (at 274.32 52.07 0)
+      (effects (font (size 1.27 1.27)) hide)
+    )
+    (property "Datasheet" "~" (id 3) (at 274.32 52.07 0)
+      (effects (font (size 1.27 1.27)) hide)
+    )
+    (pin "1")
+  )
   (symbol (lib_id "Switch:SW_DIP_x01") (at 143.51 137.16 270) (unit 1)
     (in_bom yes) (on_board yes) (fields_autoplaced)
@@
   )
   (symbol_instances
+    (path "/a6f3e91e-3057-4b03-bd5f-d7d95ebef167"
+      (reference "#FLG0101") (unit 1) (value "PWR_FLAG") (footprint "")
+    )
+    (path "/1e516542-d99b-4e7b-9506-6d9102a84b4b"
+      (reference "#FLG0102") (unit 1) (value "PWR_FLAG") (footprint "")
+    )
+    (path "/ca86c58b-c7fb-467d-a316-47a0b96c4edf"
+      (reference "#FLG0103") (unit 1) (value "PWR_FLAG") (footprint "")
+    )
     (path "/71b4e65e-9787-4d1d-be22-28dc0564d248"
       (reference "#PWR0101") (unit 1) (value "GND") (footprint "")
