File: hardware/seeq.kicad_pcb (KiCad board)
At the start: 2 copper layers, 199.5 x 82 mm, 98 parts, among them J1 MIDI IN, J2 AudioJack2, J3 Conn_01x06, J4 Conn_01x04, J5 AudioJack2, J6 MIDI OUT, SW1 SW_DIP_x01, SW10 SW_DIP_x01, SW11 SW_DIP_x01, SW12 SW_DIP_x01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

Commit message: Add jlc order number
Parts:
- moved G*** 4.45 mm to (128.7, 70.2)
Changed lines of the file:
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@@
   )
   (footprint "mod:logo-big" (layer "B.Cu")
-    (at 128.651 74.676 180)
+    (at 128.651 70.231 180)
     (attr board_only exclude_from_pos_files exclude_from_bom)
     (fp_text reference "G***" (at 0 0) (layer "B.SilkS")
@@
     (effects (font (size 2 2) (thickness 0.3)) (justify mirror))
   )
+  (gr_text "JLCJLCJLCJLC" (at 214.503 56.007) (layer "B.SilkS")
+    (effects (font (size 1 1) (thickness 0.15)) (justify mirror))
+  )
   (gr_text "${VERSION}" (at 139.954 96.647) (layer "B.SilkS")
